Commit message: img and move node

File: models/mybot/temp.urdf (robot description, URDF)
Before this commit: robot mybot, 7 links, 6 joints
Joints:
- joint camera_joint: limit lower=3.14159265359/2 upper=3.14159265359/2 effort=10 velocity=3 -> lower=-1.57079632679 upper=1.57079632679 effort=10 velocity=3; origin xyz=0.085 0 0.085 rpy=0 0 0 -> xyz=0.1 0 0.175 rpy=0 0 0; type revolute -> continuous
